File: pcb/F4/project.kicad_pcb (KiCad board)
At the start: 4 copper layers, 43 x 40.1 mm, 85 parts, among them u1 Comment, u2 Comment, u3 Comment, u4 Comment, u5 Comment, u6 Comment, u7 Comment

Commit message: PCB and CAD files updated
Parts:
- removed the ? at (146.2, 119.7)
- removed the ? at (150.2, 119.7)
- removed the ? at (148.2, 119.7)
- removed the ? at (151.2, 119.7)
- removed the ? at (147.2, 119.7)
- removed the ? at (152.2, 119.7)
- removed the ? at (149.2, 119.7)
- removed the ? at (129.5, 101.7)
- removed the ? at (128.0, 114.3)
- removed the c10 at (144.7, 120.9)
- removed the c10 at (140.3, 105.6)
- removed the c11 at (153.0, 90.2)
- removed the c11 at (138.1, 107.1)
- removed the c12 at (153.2, 107.2)
- removed the c12 at (152.9, 96.7)
- removed the r8 at (160.0, 99.0)
- removed the r8 at (157.9, 114.7)
- removed the r9 at (160.0, 101.3)
- removed the r9 at (155.7, 114.6)
- removed u4: Comment, PcbLib1:w25q
- added ?: , , F.Cu at (132.4, 99.7)
- added ?: , , F.Cu at (149.2, 119.4)
- added ?: , , F.Cu at (131.0, 102.5)
- added ?: , , F.Cu at (129.4, 112.5)
- added ?: , , F.Cu at (150.2, 119.4)
- added ?: , , F.Cu at (152.2, 119.4)
- added ?: , , F.Cu at (151.2, 119.4)
- added ?: , , F.Cu at (147.2, 119.4)
- added ?: , , F.Cu at (132.4, 96.8)
- added ?: , , F.Cu at (128.5, 102.5)
- added ?: , , F.Cu at (146.2, 119.4)
- added ?: , , F.Cu at (129.4, 115.0)
- added ?: , , F.Cu at (148.2, 119.4)
- added c10: Comment, PcbLib1:0603, F.Cu at (144.9, 100.8)
- added c11: Comment, PcbLib1:0603, F.Cu at (147.1, 101.5)
- added c12: Comment, PcbLib1:0603, F.Cu at (153.4, 89.5)
- added c26: Comment, PcbLib1:0603, B.Cu at (155.2, 97.0)
- added c27: Comment, PcbLib1:0603, B.Cu at (154.4, 100.6)
- added c28: Comment, PcbLib1:0603, B.Cu at (157.4, 109.5)
- added l1: Comment, PcbLib1:0603, B.Cu at (153.3, 90.6)
- added l2: Comment, PcbLib1:0603, B.Cu at (159.2, 90.6)
- added r10: Comment, PcbLib1:0603, F.Cu at (151.5, 123.7)
- added r11: Comment, PcbLib1:0603, B.Cu at (129.2, 118.7)
- added r12: Comment, PcbLib1:0603, B.Cu at (142.3, 103.6)
- added r13: Comment, PcbLib1:0603, B.Cu at (152.5, 105.4)
- added r14: Comment, PcbLib1:0603, B.Cu at (153.7, 116.3)
- added r15: Comment, PcbLib1:0603, B.Cu at (155.9, 116.4)
- added r16: Comment, PcbLib1:0603, B.Cu at (158.6, 106.3)
- added r17: Comment, PcbLib1:0603, B.Cu at (158.1, 115.2)
- added r18: Comment, PcbLib1:0603, B.Cu at (161.3, 96.1)
- added r19: Comment, PcbLib1:0603, B.Cu at (161.2, 98.5)
- added r2: Comment, PcbLib1:0603, F.Cu at (139.2, 94.7)
- added r20: Comment, PcbLib1:0603, B.Cu at (161.2, 100.8)
- added r8: Comment, PcbLib1:0603, F.Cu at (152.7, 103.2)
- added r9: Comment, PcbLib1:0603, F.Cu at (152.8, 105.4)
- added u8: Comment, PcbLib1:DPS368, B.Cu at (152.2, 109.4)
- c15, c16, led4, led5, pwr: moved to F.Cu
- u2: footprint PcbLib1:lqfp100 -> PcbLib1:lqfp64
- u5: footprint PcbLib1:qmc5883l -> PcbLib1:w25q; moved to F.Cu
- u6: footprint PcbLib1:icm42688 -> PcbLib1:qmc5883l
- u7: footprint PcbLib1:DPS368 -> PcbLib1:icm42688
- moved c17 29.4 mm to (132.4, 94.5)
- moved c24 26.6 mm to (155.0, 92.6)
- moved c14 24.3 mm to (150.5, 113.1), turned to -90 degrees
- moved c25 22.8 mm to (155.2, 94.8), turned to 90 degrees
- moved r4 21.7 mm to (141.3, 100.6), turned to 0 degrees
- moved c15 19.8 mm to (153.3, 112.4), turned to 180 degrees
- moved c18 18.6 mm to (133.5, 115.7)
- moved u7 12.4 mm to (149.1, 105.0), turned to 180 degrees
- moved u5 11.3 mm to (158.1, 109.1), turned to 0 degrees
- moved r5 9.56 mm to (138.5, 120.1), turned to 180 degrees
- moved c16 9.08 mm to (159.2, 92.6), turned to 90 degrees
- moved r1 7.87 mm to (139.1, 90.6)
- moved c13 7.87 mm to (153.7, 96.0), turned to 90 degrees
- moved c4 7.45 mm to (132.0, 105.5), turned to 0 degrees
- moved r3 6.80 mm to (141.7, 96.7)
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Connections:
- ? pad 1: vin -> vcc
- c13 pad 1: vcc -> xtal_out
- c14 pad 1: ant -> vcc
- c15 pad 1: gnd -> vcc
- c16 pad 1: gnd -> ant
- c18 pad 1: vcc -> gnd
- c19 pad 1: qmc_c1 -> qmc_setc
- c2 pad 1: vcc -> vbat
- c20 pad 1: qmc_setc -> qmc_c1
- c3 pad 1: osc_in -> osc_out
- c4 pad 1: osc_out -> osc_in
- c5 pad 1: vcc -> nrst
- c6 pad 1: nrst -> vcc
- c8 pad 1: vcc -> vcap1
- c9 pad 1: vcap2 -> vcc
- i2c pad 1: pd9 -> sda
- led4 pad 1: led4 -> led4r
- led5 pad 1: led5 -> led5r
- pwr pad 1: vcc -> led3r
- r1 pad 1: boot -> gnd
- r3 pad 1: gnd -> rx1
- r4 pad 1: v2_2 -> tx1
- r5 pad 1: v2_1 -> v2_2
- r7 pad 1: gnd -> vcc
- u2 pad 1: led1 -> sck2
- u5 pad 1: qmc_setc -> vcc
- u6 pad 1: gnd -> qmc_setc
Routing:
- net pa4: track 0.00 -> 53.4 mm, vias 0 -> 1
- net ch5: track 0.00 -> 52.1 mm, vias 0 -> 2
- net ch6: track 0.00 -> 49.5 mm, vias 0 -> 2
- net pc10: track 0.00 -> 43.2 mm
- net vcc: track 118.4 -> 155.9 mm, vias 19 -> 21
- net pa15: track 0.00 -> 36.7 mm
- net pb15: track 0.00 -> 34.8 mm, vias 0 -> 2
- net sck: track 37.1 -> 71.0 mm, vias 3 -> 2
- net sck2: track 13.9 -> 45.1 mm
- net miso: track 26.7 -> 57.6 mm, vias 2 -> 3
- net led4: track 46.3 -> 76.2 mm, vias 1 -> 2
- net cs4: track 2.38 -> 32.0 mm, vias 1 -> 2
- net led5: track 40.1 -> 66.8 mm, vias 1 -> 2
- net sck4: track 25.9 -> 0.00 mm, vias 2 -> 0
- net mosi4: track 25.4 -> 0.00 mm, vias 2 -> 0
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Other:
- board text added: "boot"
- board text added: "reset"
- board text added: "v"
- board text removed: "5v"
- board text removed: "bt"
- board text removed: "rst"
