File: pcb/H7/esp8285.kicad_sch (KiCad schematic)
At the start: 12 parts, among them U26 ESP8266EX

Commit message: H7 schematic updated
Parts:
- renumbered C19 to C20, C20 to C21, C28 to C27, R12 to R10, U26 to U1
Changed lines of the file:
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@@
 		(on_board yes)
 		(dnp no)
-		(property "Reference" "C20"
+		(property "Reference" "C21"
 			(at 118.11 85.344 0)
 			(effects
@@
 			(project "project"
 				(path "/b61a0d2b-7633-4d0a-8bfd-ad16aaa1ff64/b2e80637-8828-4221-a6bd-d0ac0b787eac"
-					(reference "C20")
+					(reference "C21")
 					(unit 1)
 				)
@@
 		(dnp no)
 		(fields_autoplaced yes)
-		(property "Reference" "R12"
+		(property "Reference" "R10"
 			(at 146.05 83.82 90)
 			(effects
@@
 			(project "project"
 				(path "/b61a0d2b-7633-4d0a-8bfd-ad16aaa1ff64/b2e80637-8828-4221-a6bd-d0ac0b787eac"
-					(reference "R12")
+					(reference "R10")
 					(unit 1)
 				)
@@
 		(on_board yes)
 		(dnp no)
-		(property "Reference" "U26"
+		(property "Reference" "U1"
 			(at 163.576 125.73 0)
 			(effects
@@
 			(project "project"
 				(path "/b61a0d2b-7633-4d0a-8bfd-ad16aaa1ff64/b2e80637-8828-4221-a6bd-d0ac0b787eac"
-					(reference "U26")
+					(reference "U1")
 					(unit 1)
 				)
@@
 		(on_board yes)
 		(dnp no)
-		(property "Reference" "C28"
+		(property "Reference" "C27"
 			(at 128.27 85.344 0)
 			(effects
@@
 			(project "project"
 				(path "/b61a0d2b-7633-4d0a-8bfd-ad16aaa1ff64/b2e80637-8828-4221-a6bd-d0ac0b787eac"
-					(reference "C28")
+					(reference "C27")
 					(unit 1)
 				)
@@
 		(on_board yes)
 		(dnp no)
-		(property "Reference" "C19"
+		(property "Reference" "C20"
 			(at 107.442 85.344 0)
 			(effects
@@
 			(project "project"
 				(path "/b61a0d2b-7633-4d0a-8bfd-ad16aaa1ff64/b2e80637-8828-4221-a6bd-d0ac0b787eac"
-					(reference "C19")
-					(unit 1)
-				)
+					(reference "C20")
+					(unit 1)
+				)

Commit message: schematic updated
Parts:
- removed C4: 5.6pF, symbol Device:C
- added L1: tbd, symbol Device:L
- R9: renamed from R10; value R -> 12kΩ
- renumbered C27 to C18, C21 to C24, C20 to C29, L1 to C5, L2 to C6, C5 to C7, C6 to C8
Connections:
- net LDA is gone; now on net LNA: U1.2 (LNA)
- net LNA: now also L1.2; no longer C5.2
- net at AE1.1 (A): now also C5.2, L1.1
- net PB5 renamed GPIO_EXTI7
- net PB6 renamed GPIO_BOOT
- net PB7 renamed GPIO_BUSY
- net PC2 renamed SPI2_MISO
- net PC3 renamed SPI2_MOSI
- net PD3 renamed SPI2_SCK
- net PE0 renamed SPI2_NSS
- net PE1 renamed GPIO_EXTRSTB
Other:
- moved on the sheet: C5, R9
