File: pcb/H7/project.kicad_sch (KiCad schematic)
At the start: 61 parts, among them J3 bt, J4 rst, U11 STM32H723VGT6, U14 TPS5430DDAR, U17 LDL1117S33R, U23 W25Q128FVSIG

Commit message: H7 schematic updated
Parts:
- removed C21: 4.7uF, symbol Device:C
- removed U21: ~, symbol library:QMC5883L
- added C7: 0.1uF, symbol Device:C
- added U6: LIS3MDL, Package_LGA:LGA-12_2x2mm_P0.5mm, symbol Sensor_Magnetic:LIS3MDL
- C29: renamed from C22; value 0.22uF -> 1uF
- D7: value LED1 -> LED2
- D8: value LED2 -> LED1
- R5: value 3kΩ -> 5.1kΩ
- U5: renamed from U18; value ~ -> DPS368XTSA1
- U7: renamed from U13; value ~ -> ICM-42688-P
- renumbered C37 to C10, C10 to C11, C11 to C12, C12 to C13, C13 to C14, C14 to C15, C15 to C16, C16 to C17, C17 to C18, C18 to C19, C23 to C22, C24 to C23, C25 to C24, C26 to C25, C27 to C26, C29 to C28, C50 to C32, C7 to C8, C8 to C9, R17 to R9, U11 to U2, U17 to U3, U14 to U4, U23 to U8
Connections:
- net +3.3V: now also C29.2, U6.10 (~{CS}), U6.5 (Vdd), U6.6 (Vdd_IO)
- net GND: now also C29.1, C30.2, C7.2, U6.12 (GND), U6.2 (GND), U6.3 (GND), U6.9 (SDO/SA1)
- net PB11: now also R11.1
- net PB12: now also R10.1; no longer R11.1
- net PB13: no longer R10.1
- net PB3: no longer U8.6 (CLK)
- net PB4: no longer U8.2 (DO/IO_{1})
- net PB8: now also U6.1 (SCL/SPC)
- net PB9: now also U6.11 (SDA/SDI/SDO)
- net PD4: now also U6.8 (DRDY)
- net PD7: no longer U8.5 (DI/IO_{0})
- new net: C7.1, U6.4 (C1)
- new net PA5: U8.6 (CLK)
- new net PA6: U8.2 (DO/IO_{1})
- new net PA7: U8.5 (DI/IO_{0})
Other:
- moved on the sheet: C29, C30

Commit message: schematic updated
Parts:
- removed C28: 4.7uF, symbol Device:C
- removed C8: 1uF, symbol Device:C
- removed U3: LDL1117S33R, Package_TO_SOT_SMD:SOT-223-3_TabPin2, symbol Regulator_Linear:AMS1117-3.3
- added C10, C3: 1uF, symbol Device:C
- added C12: 10uF, symbol Device:C
- added C13: 47uF, symbol Device:C
- added R10, R11, R12, R13, R14, R17, R18, R21: 33Ω, symbol Device:R
- added R19: 47Ω, symbol Device:R
- added U3: TPS7A4700, Package_DFN_QFN:Texas_RGW0020A_VQFN-20-1EP_5x5mm_P0.65mm_EP3.15x3.15mm_ThermalVias, symbol Regulator_Linear:TPS7A4701xRGW
- added U9: ~, symbol library:CRSF
- J3: value bt -> boot
- R5: value 5.1kΩ -> 680Ω
- R6: value 680Ω -> 5.1kΩ
- cr1: value 20 mHz -> 20mHz
- renumbered C9 to C11, C10 to C14, C12 to C15, C11 to C16, C26 to C17, C30 to C19, C29 to C20, C32 to C21, C33 to C22, C3 to C23, C22 to C25, C24 to C26, C25 to C27, C23 to C28, C18 to C30, C19 to C31, C31 to C32, C14 to C33, C13 to C34, C16 to C35, C17 to C36, C15 to C4, C7 to C9, D1 to D2, L3 to L2, R8 to R15, R9 to R16, R3 to R5
Connections:
- net +3.3V: now also C13.1, C3.2, R19.1, U3.1 (OUT), U3.20 (OUT), U3.3 (SENSE/FB); no longer U2.20 (VREF+)
- net +5V: now also C12.1, U3.13 (EN), U3.15 (IN), U3.16 (IN), U9.3 (5v)
- net GND: now also C10.1, C12.2, C13.2, C3.1, U3.11 (0.2V), U3.12 (0.1V), U3.21 (EP), U3.7 (GND), U3.8 (1.6V), U9.4 (GND)
- net GPIO_EXTI0: now reaches U5.5 (SDO)
- net GPIO_EXTI0: now also U2.22 (PA0)
- net at U2.28 (PA4): now also R12.2
- net at U2.29 (PA5): now also R11.2
- net at U2.30 (PA6): now also R10.2
- net at U2.31 (PA7): now also R13.2
- net UART1_TX: now reaches U2.53 (PB14)
- net UART1_TX: now also U9.1 (TX)
- net UART1_RX: now reaches U2.54 (PB15)
- net UART1_RX: now also U9.2 (RX)
- net SPI1_NSS: now reaches U2.77 (PA15(JTDI))
- net SPI1_NSS: now also U7.12 (AP_CS)
- net PA10 renamed TIM1_CH3
- net PA11 renamed TIM1_CH4
- net PA12 renamed GPIO_FSYNC
- net PA13 renamed SWD_DIO
- net PA14 renamed SWD_CLK
- net PA5 renamed SPI6_SCK
- net SPI6_SCK: now also R11.1
- net PA6 renamed SPI6_MISO
- net SPI6_MISO: now also R10.1
- net PA7 renamed SPI6_MOSI
- net SPI6_MOSI: now also R13.1
- net PA8 renamed TIM1_CH1
- net PA9 renamed TIM1_CH2
- net PB10 renamed UART3_TX
- net PB11 renamed UART3_RX
- net UART3_RX: no longer R11.1
- net PB12 renamed GPIO_LED1
- net PB13 renamed GPIO_LED2
- net GPIO_LED2: now also R11.1
- net PB3 renamed SPI1_SCK
- net PB4 renamed SPI1_MISO
- net PB5 renamed SPI1_MOSI
- net SPI1_MOSI: now also U7.14 (AP_SDI)
- net PB6 renamed I2C1_SCL
- net I2C1_SCL: now also R1.2, U19.4 (SCL), U5.4 (SCK), U6.1 (SCL/SPC)
- net PB7 renamed I2C1_SDA
- net I2C1_SDA: now also R7.1, U19.5 (SDA), U5.3 (SDI), U6.11 (SDA/SDI/SDO)
- removed net PB8: R1.2, U19.4 (SCL), U2.95 (PB8), U5.4 (SCK), U6.1 (SCL/SPC)
- removed net PB9: R7.1, U19.5 (SDA), U2.96 (PB9), U5.3 (SDI), U6.11 (SDA/SDI/SDO)
- net PC10: no longer names the net of U2.78 (PC10)
- net PC10: no longer U8.1 (~{CS})
- net PC11: no longer names the net of U2.79 (PC11)
- net PC11: no longer U7.12 (AP_CS)
- net PC12 renamed UART5_TX
- net PC2: no longer names the net of U2.17 (PC2_C)
- net PC2: now also R18.1
- net PC3: no longer names the net of U2.18 (PC3_C)
- net PC3: now also R21.1
- net PC4 renamed ADC1_INP4
- net PC5 renamed ADC2_INP8
- net PD0 renamed UART4_RX
- net PD1 renamed UART4_TX
- net PD2 renamed UART5_RX
- net PD3: no longer names the net of U2.84 (PD3)
- net PD3: now also R14.1
- net PD4 renamed GPIO_EXTI4
- net PD5 renamed UART2_TX
- net PD6 renamed UART2_RX
- net PD7 renamed GPIO_EXTI7
- net GPIO_EXTI7: no longer U7.14 (AP_SDI)
- net PE0 renamed GPIO_BUSY
- net PE1 renamed GPIO_EXTRSTB
- net PE2 renamed SPI4_SCK
- net PE3 renamed GPIO_EXTI3
- net PE4 renamed SPI4_NSS
- net PE5 renamed SPI4_MISO
- net PE6 renamed SPI4_MOSI
- new net: C10.2, U3.14 (NR)
- new net: R17.1, U2.96 (PB9)
- new net GPIO_BOOT: U2.95 (PB8)
- new net SPI2_MISO: R18.2
- new net SPI2_MOSI: R21.2
- new net SPI2_NSS: R17.2
- new net SPI2_SCK: R14.2
- new net SPI6_NSS: R12.1, U8.1 (~{CS})
- new net VREF+: R19.2, U2.20 (VREF+)
- no-connect marks 42 -> 45
Other:
- note added: "LIDAR"
- note removed: "LDO"
- moved on the sheet: C1, C11, C14, C15, C16, C17, C2, C21, C22, C23, C25, C26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
